File: PROJECT/MACH/MACH_THUC/MACH_THUC/MACH_THUC/MACH_THUC.kicad_pcb (KiCad board)
At the start: 2 copper layers, 30 parts, among them Q1 2SB688, U1 LM7805_TO220

Commit message: update code
Parts:
- added C8: 33pF, library_thuan_footprint:CAP_104, F.Cu at (185.3, 120.7)
- added C9: 33pF, library_thuan_footprint:CAP_104, F.Cu at (193.9, 120.7)
- added CR1: ~, library_thuan_footprint:cr2032, F.Cu at (174.0, 100.5)
- added D4: LED-RELAY_1, library_thuan_footprint:LED_5MM, F.Cu at (130.8, 111.8)
- added D5: 1N4007, library_thuan_footprint:1N4007, F.Cu at (103.8, 56.2)
- added D6: LED-RELAY_1, library_thuan_footprint:LED_5MM, F.Cu at (111.8, 118.0)
- added D7: 1N4007, library_thuan_footprint:1N4007, F.Cu at (86.4, 57.3)
- added DDS18B20: ~, library_thuan_footprint:DOMINO_3, F.Cu at (262.2, 151.4)
- added ESP_12E1: ~, library_thuan_footprint:ESP8266_12E, F.Cu at (200.3, 92.8)
- added K1: SANYOU_SRD_Form_C, Relay_THT:Relay_SPDT_SANYOU_SRD_Series_Form_C, F.Cu at (104.1, 58.0)
- added K2: SANYOU_SRD_Form_C, Relay_THT:Relay_SPDT_SANYOU_SRD_Series_Form_C, F.Cu at (81.6, 57.8)
- added Q2: BC547, Package_TO_SOT_THT:TO-92_Inline, F.Cu at (81.3, 69.8)
- added Q3: BC547, Package_TO_SOT_THT:TO-92_Inline, F.Cu at (98.8, 68.8)
- added R10: 4.7k, library_thuan_footprint:RES_DEFAULT, F.Cu at (166.7, 77.1)
- added R11: 4.7k, library_thuan_footprint:RES_DEFAULT, F.Cu at (166.8, 85.2)
- added R12: 4.7k, library_thuan_footprint:RES_DEFAULT, F.Cu at (229.9, 104.4)
- added R13: 1.2k, library_thuan_footprint:RES_DEFAULT, F.Cu at (214.1, 79.8)
- added R14: 2.4k, library_thuan_footprint:RES_DEFAULT, F.Cu at (214.1, 84.0)
- added R15: 1k, library_thuan_footprint:RES_DEFAULT, F.Cu at (120.8, 94.2)
- added R16: 330, library_thuan_footprint:RES_DEFAULT, F.Cu at (124.6, 94.3)
- added R17: 1k, library_thuan_footprint:RES_DEFAULT, F.Cu at (97.0, 72.6)
- added R18: 1k, library_thuan_footprint:RES_DEFAULT, F.Cu at (101.8, 100.3)
- added R19: 330, library_thuan_footprint:RES_DEFAULT, F.Cu at (105.6, 100.4)
- added R20: 1k, library_thuan_footprint:RES_DEFAULT, F.Cu at (80.2, 73.7)
- added RV1: 10k, library_thuan_footprint:RM065-103, F.Cu at (254.9, 28.1)
- added SERVO1: ~, library_thuan_footprint:DOMINO_3, F.Cu at (262.2, 140.1)
- added U2: DS1307+, Package_DIP:DIP-8_W7.62mm, F.Cu at (152.8, 97.0)
- added U3: LCD-016N002L, Display:LCD-016N002L, F.Cu at (198.1, 30.2)
- added U4: PCF8574, library_thuan_footprint:PCF8574, F.Cu at (223.5, 53.5)
- added U5: PC817, Package_DIP:DIP-4_W7.62mm, F.Cu at (129.5, 87.8)
- added U6: PC817, Package_DIP:DIP-4_W7.62mm, F.Cu at (110.5, 92.7)
- added Y1: Crystal 20M, library_thuan_footprint:crytal_20M, F.Cu at (188.6, 128.5)
- added Y2: Crystal 32.768KHz, library_thuan_footprint:crytal_32.768KHz, F.Cu at (153.5, 110.8)
- added d3r1: ~, library_thuan_footprint:DOMINO_3, F.Cu at (106.4, 24.3)
- added d3r2: ~, library_thuan_footprint:DOMINO_3, F.Cu at (83.8, 24.1)
- moved PIC16F877A1 247.8 mm to (254.0, 119.5), turned to -90 degrees
- moved PB1 214.5 mm to (207.3, 136.2)
- moved PB2 212.5 mm to (216.1, 136.2)
- moved PB3 210.4 mm to (224.8, 136.2)
- moved PB4 208.4 mm to (233.5, 136.2)
- moved PB5 206.4 mm to (242.2, 136.2)
- moved D3 204.0 mm to (176.5, 143.7)
- moved R4 193.5 mm to (187.2, 146.2), turned to -90 degrees
- moved R5 193.5 mm to (207.3, 130.4)
- moved R6 193.5 mm to (216.0, 130.4)
- moved R7 193.5 mm to (224.7, 130.4)
- moved R8 193.5 mm to (233.4, 130.4)
- moved R9 193.5 mm to (242.2, 130.4)
- moved C5 163.7 mm to (181.3, 146.5), turned to -90 degrees
- moved R2 147.6 mm to (153.6, 141.1), turned to -90 degrees
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Connections:
- PIC16F877A1 pad 1: unconnected-(PIC16F877A1-MCLR-Pad1) -> rst
- PIC16F877A1 pad 11: unconnected-(PIC16F877A1-VDD-Pad11) -> +5V
- PIC16F877A1 pad 12: unconnected-(PIC16F877A1-VSS-Pad12) -> GND1
- PIC16F877A1 pad 13: unconnected-(PIC16F877A1-OSC1/CLKI-Pad13) -> osc1
- PIC16F877A1 pad 14: unconnected-(PIC16F877A1-OSC2/CLK0-Pad14) -> osc2
- PIC16F877A1 pad 16: unconnected-(PIC16F877A1-RC1/CCP2-Pad16) -> servo
- PIC16F877A1 pad 18: unconnected-(PIC16F877A1-RC3/SCL-Pad18) -> scl
- PIC16F877A1 pad 2: unconnected-(PIC16F877A1-RA0/AN0-Pad2) -> ds_18b20
- PIC16F877A1 pad 23: unconnected-(PIC16F877A1-RC4/SDA-Pad23) -> sda
- PIC16F877A1 pad 25: unconnected-(PIC16F877A1-RC6-Pad25) -> tx
- PIC16F877A1 pad 26: unconnected-(PIC16F877A1-RC7-Pad26) -> rx
- PIC16F877A1 pad 29: unconnected-(PIC16F877A1-RD6-Pad29) -> relay_2
- PIC16F877A1 pad 30: unconnected-(PIC16F877A1-RD7-Pad30) -> relay_1
- PIC16F877A1 pad 31: unconnected-(PIC16F877A1-VSS-Pad31) -> GND1
- PIC16F877A1 pad 32: unconnected-(PIC16F877A1-VDD-Pad32) -> +5V
- PIC16F877A1 pad 33: unconnected-(PIC16F877A1-RB0-Pad33) -> btn_1
- PIC16F877A1 pad 34: unconnected-(PIC16F877A1-RB1-Pad34) -> btn_2
- PIC16F877A1 pad 35: unconnected-(PIC16F877A1-RB2-Pad35) -> btn_3
- PIC16F877A1 pad 36: unconnected-(PIC16F877A1-RB3-Pad36) -> btn_4
Routing:
- net GND1: track 0.00 -> 723.4 mm, vias 0 -> 2
- net +5V: track 0.00 -> 614.7 mm, vias 0 -> 4
- net +5P: track 0.00 -> 222.0 mm, vias 0 -> 4
- net sda: track 0.00 -> 167.2 mm, vias 0 -> 2
- net Net-(B1-VIN): track 0.00 -> 150.7 mm
- net relay_2: track 0.00 -> 133.9 mm, vias 0 -> 2
- net scl: track 0.00 -> 130.8 mm, vias 0 -> 2
- net Net-(D1-A): track 0.00 -> 129.9 mm, vias 0 -> 2
- net relay_1: track 0.00 -> 112.6 mm, vias 0 -> 2
- net GND2: track 0.00 -> 109.2 mm, vias 0 -> 2
- net servo: track 0.00 -> 97.0 mm, vias 0 -> 2
- net Net-(U3-DB7): track 0.00 -> 84.1 mm
- net Net-(U3-DB6): track 0.00 -> 75.4 mm
- net ds_18b20: track 0.00 -> 70.1 mm, vias 0 -> 2
- net rst: track 0.00 -> 69.5 mm
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Other:
- board outline added: 204.5 x 138.6 mm

Commit message: update code
Parts:
- removed D2: 1N4007, library_thuan_footprint:1N4007
- added C10: 100nF, library_thuan_footprint:CAP_104, F.Cu at (174.0, 140.2)
- added C6P1: ~, library_thuan_footprint:CONNECT_6PIN, F.Cu at (61.0, 128.3)
- C8, C9: value 33pF -> 22pF
- d3r1: footprint library_thuan_footprint:DOMINO_3 -> library_thuan_footprint:DOMINO_3_5mm
- d3r2: footprint library_thuan_footprint:DOMINO_3 -> library_thuan_footprint:DOMINO_3_5mm; moved to B.Cu
- domino4P1: footprint library_thuan_footprint:DOMINO_4 -> library_thuan_footprint:DOMINO_4_5mm
- moved DDS18B20 213.1 mm to (50.8, 124.5), turned to -90 degrees
- moved SERVO1 211.5 mm to (50.8, 135.7), turned to -90 degrees
- moved RV1 181.8 mm to (85.1, 93.0)
- moved PIC16F877A1 160.1 mm to (94.1, 113.0), turned to 90 degrees
- moved C8 137.2 mm to (49.5, 100.4)
- moved C9 137.2 mm to (58.2, 100.4)
- moved Y1 132.9 mm to (57.1, 108.7)
- moved R12 115.7 mm to (118.5, 73.2)
- moved C7 103.3 mm to (43.5, 79.2)
- moved C5 99.0 mm to (84.1, 127.6), turned to 0 degrees
- moved R4 95.6 mm to (118.1, 80.2), turned to 0 degrees
- moved C4 95.0 mm to (72.4, 130.9), turned to 0 degrees
- moved R16 87.6 mm to (37.0, 94.0)
- moved D4 87.5 mm to (45.7, 91.4), turned to 0 degrees
- moved R13 87.2 mm to (127.2, 73.2)
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Connections:
- PIC16F877A1 pad 39: unconnected-(PIC16F877A1-RB6-Pad39) -> pgc
- PIC16F877A1 pad 40: unconnected-(PIC16F877A1-RB7-Pad40) ->  pgd
- U1 pad 2: Net-(D2-A) -> GND1
Routing:
- net GND1: track 723.4 -> 478.6 mm, vias 2 -> 0
- net +5V: track 614.7 -> 391.0 mm, vias 4 -> 0
- net +5P: track 222.0 -> 124.8 mm, vias 4 -> 0
- net btn_4: track 23.5 -> 120.0 mm
- net btn_3: track 25.3 -> 106.8 mm
- net relay_2: track 133.9 -> 63.6 mm, vias 2 -> 0
- net rst: track 69.5 -> 139.7 mm, vias 0 -> 1
- net btn_2: track 30.8 -> 93.5 mm
- net pgc: track 0.00 -> 60.1 mm, vias 0 -> 1
- net  pgd: track 0.00 -> 56.4 mm
- net osc2: track 51.3 -> 99.2 mm
- net btn_1: track 35.2 -> 83.0 mm, vias 0 -> 1
- net Net-(U3-DB7): track 84.1 -> 37.2 mm
- net ds_18b20: track 70.1 -> 115.2 mm, vias 2 -> 1
- net Net-(ESP_12E1-RX): track 30.0 -> 73.8 mm
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Other:
- board size 204.5 x 138.6 mm -> 177.8 x 99.1 mm

Commit message: update code
Connections:
- R16 pad 2: Net-(R16-Pad2) -> GND1
- R19 pad 2: Net-(R19-Pad2) -> GND1
- U5 pad 2: Net-(R16-Pad2) -> GND1
- U6 pad 2: Net-(R19-Pad2) -> GND1
Routing:
- net GND1: track 478.6 -> 530.3 mm
- net Net-(R19-Pad2): track 8.68 -> 0.00 mm
- net Net-(R16-Pad2): track 8.68 -> 0.00 mm

Commit message: update code'
Parts:
- U4: footprint library_thuan_footprint:PCF8574 -> library_thuan_footprint:SOIC127P1032X265-16N
- d3r2: moved to F.Cu
- moved SERVO1 157.8 mm to (207.0, 113.0), turned to 90 degrees
- moved DDS18B20 156.2 mm to (207.0, 124.3), turned to 90 degrees
- moved R15 118.8 mm to (154.9, 61.1), turned to 0 degrees
- moved CR1 113.0 mm to (201.8, 119.4)
- moved U5 110.3 mm to (158.8, 119.4)
- moved Y1 106.0 mm to (155.7, 69.6)
- moved Q2 105.1 mm to (160.0, 130.8)
- moved Q3 94.9 mm to (168.9, 130.8)
- moved R20 91.2 mm to (145.9, 66.2)
- moved C7 89.2 mm to (132.7, 78.2), turned to 90 degrees
- moved C8 88.7 mm to (136.6, 83.8), turned to 90 degrees
- moved R10 86.1 mm to (111.3, 61.1)
- moved R11 86.1 mm to (120.1, 61.1)
- moved C6 82.2 mm to (132.5, 83.8), turned to 90 degrees
- moved U6 81.8 mm to (151.1, 127.0), turned to 90 degrees
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Connections:
- ESP_12E1 pad 18: rx -> unconnected-(ESP_12E1-TX-Pad18)
- ESP_12E1 pad 19: Net-(ESP_12E1-RX) -> unconnected-(ESP_12E1-RX-Pad19)
- ESP_12E1 pad 20: unconnected-(ESP_12E1-D8-Pad20) -> rx
- ESP_12E1 pad 21: unconnected-(ESP_12E1-D7-Pad21) -> Net-(ESP_12E1-D7)
- R13 pad 2: Net-(ESP_12E1-RX) -> Net-(ESP_12E1-D7)
- R14 pad 1: Net-(ESP_12E1-RX) -> Net-(ESP_12E1-D7)
- U3 pad 15: Net-(U3-A/VEE) -> +5V
- U4 pad 7: Net-(U3-A/VEE) -> unconnected-(U4-P3-Pad7)
Routing:
- net ds_18b20: track 115.2 -> 247.0 mm, vias 1 -> 0
- net Net-(D7-A): track 13.9 -> 132.0 mm, vias 0 -> 1
- net Net-(D5-A): track 14.0 -> 125.5 mm, vias 0 -> 1
- net Net-(Q3-B): track 7.40 -> 107.2 mm
- net +5V: track 391.0 -> 484.8 mm, vias 0 -> 1
- net Net-(R17-Pad1): track 16.7 -> 100.3 mm, vias 0 -> 1
- net scl: track 113.3 -> 191.3 mm, vias 0 -> 1
- net Net-(ESP_12E1-RX): track 73.8 -> 0.00 mm
- net servo: track 99.7 -> 173.4 mm, vias 0 -> 1
- net tx: track 33.7 -> 101.0 mm, vias 0 -> 1
- net Net-(R18-Pad2): track 3.82 -> 62.1 mm
- net Net-(Q2-B): track 7.48 -> 64.4 mm
- net Net-(ESP_12E1-D7): track 0.00 -> 56.1 mm
- net Net-(D1-A): track 104.8 -> 154.3 mm, vias 1 -> 0
- net Net-(R15-Pad2): track 3.86 -> 51.7 mm
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Other:
- board outline removed
