File: PROJECT/MACH/MACH_THUC/MACH_THUC/MACH_THUC/MACH_THUC.kicad_sch (KiCad schematic)
At the start: 32 parts, among them Q1 2SB688, U1 LM7805_TO220

Commit message: update code
Parts:
- added C8, C9: 33pF, library_thuan_footprint:CAP_104, symbol Device:C
- added CR1: ~, library_thuan_footprint:cr2032, symbol library_thuan:CR2032
- added D4, D6: LED-RELAY_1, library_thuan_footprint:LED_5MM, symbol Device:LED
- added D5, D7: 1N4007, library_thuan_footprint:1N4007, symbol Device:D
- added DDS18B20, SERVO1: ~, library_thuan_footprint:DOMINO_3, symbol library_thuan:domino_3pin
- added ESP_12E1: ~, library_thuan_footprint:ESP8266_12E, symbol library_thuan:ESP8266
- added K1, K2: SANYOU_SRD_Form_C, Relay_THT:Relay_SPDT_SANYOU_SRD_Series_Form_C, symbol Relay:SANYOU_SRD_Form_C
- added Q2, Q3: BC547, Package_TO_SOT_THT:TO-92_Inline, symbol Transistor_BJT:BC547
- added R12: 4.7k, library_thuan_footprint:RES_DEFAULT, symbol Device:R
- added R13: 1.2k, library_thuan_footprint:RES_DEFAULT, symbol Device:R
- added R14: 2.4k, library_thuan_footprint:RES_DEFAULT, symbol Device:R
- added R15, R17, R18, R20: 1k, library_thuan_footprint:RES_DEFAULT, symbol Device:R
- added R16, R19: 330, library_thuan_footprint:RES_DEFAULT, symbol Device:R
- added RV1: 10k, library_thuan_footprint:RM065-103, symbol Device:R_Potentiometer
- added U2: DS1307+, Package_DIP:DIP-8_W7.62mm, symbol Timer_RTC:DS1307+
- added U3: LCD-016N002L, Display:LCD-016N002L, symbol Display_Character:LCD-016N002L
- added U4: PCF8574, library_thuan_footprint:PCF8574, symbol Interface_Expansion:PCF8574
- added U5, U6: PC817, Package_DIP:DIP-4_W7.62mm, symbol Isolator:PC817
- added Y1: Crystal 20M, library_thuan_footprint:crytal_20M, symbol Device:Crystal
- added Y2: Crystal 32.768KHz, library_thuan_footprint:crytal_32.768KHz, symbol Device:Crystal
- added d3r1, d3r2: ~, library_thuan_footprint:DOMINO_3, symbol library_thuan:domino_3_relay
Connections:
- net +5P: now also D5.1 (K), D7.1 (K), K1.5, K2.5, U5.4, U6.4
- net +5V: now also DDS18B20.3 (VCC), ESP_12E1.15 (VIN), R12.1, RV1.3, SERVO1.3 (VCC), U2.8 (VCC), U3.2 (VDD), U4.1 (A0), U4.16 (VDD), U4.2 (A1), U4.3 (A2)
- net GND1: now also C8.2, C9.2, CR1.1 (GND), DDS18B20.1 (GND), ESP_12E1.14 (G), R14.2, RV1.1, SERVO1.1 (GND), U2.4 (GND), U3.1 (VSS), U3.16 (K), U4.8 (VSS)
- net GND2: now also Q2.3 (E), Q3.3 (E)
- net ds_18b20: now also DDS18B20.2 (D), R12.2
- net osc1: now also C9.1, Y1.2
- net osc2: now also C8.1, Y1.1
- net rx: now also ESP_12E1.18 (TX)
- net scl: now also U2.6 (SCL), U4.14 (SCL)
- net sda: now also U2.5 (SDA), U4.15 (SDA)
- net servo: now also SERVO1.2 (D)
- net tx: now also R13.1
- net relay_2: now reaches PIC16F877A1.29 (RD6)
- net relay_2: now also D6.2 (A), R18.1
- net relay_1: now reaches PIC16F877A1.30 (RD7)
- net relay_1: now also D4.2 (A), R15.1
- new net: D7.2 (A), K2.2, Q2.1 (C)
- new net: Q2.2 (B), R20.2
- new net: R15.2, U5.1
- new net: R16.2, U5.2
- new net: R17.1, U5.3
- new net: ESP_12E1.19 (RX), R13.2, R14.1
- new net: Q3.2 (B), R17.2
- new net: R18.2, U6.1
- new net: R19.2, U6.2
- new net: R20.1, U6.3
- new net: U2.1 (X1), Y2.2
- new net: U2.2 (X2), Y2.1
- new net: CR1.2 (VCC), U2.3 (VBAT)
- new net: K1.1, d3r1.2 (CO)
- new net: D5.2 (A), K1.2, Q3.1 (C)
- new net: K1.3, d3r1.1 (NO)
- new net: K1.4, d3r1.3 (NC)
- new net: K2.3, d3r2.1 (NO)
- new net: K2.1, d3r2.2 (CO)
- new net: K2.4, d3r2.3 (NC)
- new net: D6.1 (K), R19.1
- new net: U3.12 (DB5), U4.10 (P5)
- new net: U3.13 (DB6), U4.11 (P6)
- new net: U3.14 (DB7), U4.12 (P7)
- new net: U3.4 (RS), U4.4 (P0)
- new net: U3.5 (R/~{W}), U4.5 (P1)
- new net: U3.6 (E), U4.6 (P2)
- new net: U3.15 (A/VEE), U4.7 (P3)
- new net: U3.11 (DB4), U4.9 (P4)
- new net: D4.1 (K), R16.1
- new net: RV1.2, U3.3 (VO)
Other:
- moved on the sheet: R10, R11

Commit message: update code
Parts:
- removed D2: 1N4007, library_thuan_footprint:1N4007, symbol Device:D
- added C10: 100nF, library_thuan_footprint:CAP_104, symbol Device:C
- added C6P1: ~, library_thuan_footprint:CONNECT_6PIN, symbol library_thuan:CONNECT_6PIN
- C8, C9: value 33pF -> 22pF
- d3r1, d3r2: footprint library_thuan_footprint:DOMINO_3 -> library_thuan_footprint:DOMINO_3_5mm
- domino4P1: footprint library_thuan_footprint:DOMINO_4 -> library_thuan_footprint:DOMINO_4_5mm
Connections:
- net +5V: now also C6P1.2
- net GND1: now also U1.2 (GND), C10.2, C6P1.3
- net rst: now also C10.1, C6P1.1
- net pgc: now reaches PIC16F877A1.39 (RB6)
- net pgc: now also C6P1.5
- net  pgd: now reaches PIC16F877A1.40 (RB7)
- net  pgd: now also C6P1.4
- no-connect marks 0 -> 2
Other:
- moved on the sheet: PB2, PB3, PB4, PB5, R5, R6, R7, R8, R9

Commit message: update code
Connections:
- net GND1: now also R16.2, R19.2, U5.2, U6.2
Other:
- moved on the sheet: R16, R19
Changed lines of the file:
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@@
   (junction (at 59.69 121.285) (diameter 0) (color 0 0 0 0)
   )
+  (junction (at 194.31 151.765) (diameter 0) (color 0 0 0 0)
+  )
   (junction (at 227.33 29.21) (diameter 0) (color 0 0 0 0)
   )
@@
   (junction (at 212.725 61.595) (diameter 0) (color 0 0 0 0)
   )
+  (junction (at 182.88 128.905) (diameter 0) (color 0 0 0 0)
+  )
   (junction (at 38.1 31.115) (diameter 0) (color 0 0 0 0)
   )
@@
     (stroke (width 0) (type default))
   )
+  (wire (pts (xy 193.675 151.765) (xy 194.31 151.765))
+    (stroke (width 0) (type default))
+  )
   (wire (pts (xy 188.595 80.01) (xy 188.595 87.63))
     (stroke (width 0) (type default))
@@
     (stroke (width 0) (type default))
   )
+  (wire (pts (xy 194.31 151.765) (xy 194.945 151.765))
+    (stroke (width 0) (type default))
+  )
   (wire (pts (xy 148.59 43.815) (xy 152.4 43.815))
     (stroke (width 0) (type default))
@@
     (stroke (width 0) (type default))
   )
+  (wire (pts (xy 182.88 128.905) (xy 183.515 128.905))
+    (stroke (width 0) (type default))
+  )
   (wire (pts (xy 48.26 51.435) (xy 48.26 60.96))
     (stroke (width 0) (type default))
@@
     (stroke (width 0) (type default))
   )
+  (wire (pts (xy 182.245 128.905) (xy 182.88 128.905))
+    (stroke (width 0) (type default))
+  )
   (wire (pts (xy 46.99 163.83) (xy 49.53 163.83))
     (stroke (width 0) (type default))
@@
     (stroke (width 0) (type default))
   )
-  (wire (pts (xy 186.055 151.765) (xy 187.325 151.765))
-    (stroke (width 0) (type default))
-  )
   (wire (pts (xy 120.015 29.21) (xy 120.015 31.115))
     (stroke (width 0) (type default))
@@
     (stroke (width 0) (type default))
   )
-  (wire (pts (xy 174.625 128.905) (xy 175.895 128.905))
-    (stroke (width 0) (type default))
-  )
   (wire (pts (xy 104.14 38.735) (xy 104.14 41.275))
     (stroke (width 0) (type default))
@@
     )
   )
-  (symbol (lib_id "Device:R") (at 191.135 151.765 90) (unit 1)
+  (symbol (lib_id "Device:R") (at 189.865 151.765 90) (unit 1)
     (in_bom yes) (on_board yes) (dnp no) (fields_autoplaced)
-    (property "Reference" "R19" (at 191.135 145.415 90)
+    (property "Reference" "R19" (at 189.865 145.415 90)
       (effects (font (size 1.27 1.27)))
     )
-    (property "Value" "330" (at 191.135 147.955 90)
+    (property "Value" "330" (at 189.865 147.955 90)
       (effects (font (size 1.27 1.27)))
     )
-    (property "Footprint" "library_thuan_footprint:RES_DEFAULT" (at 191.135 153.543 90)
+    (property "Footprint" "library_thuan_footprint:RES_DEFAULT" (at 189.865 153.543 90)
       (effects (font (size 1.27 1.27)) hide)
     )
-    (property "Datasheet" "https://www.thegioiic.com/dien-tro-330-kohm-1-4w-5-4-vong-mau" (at 191.135 151.765 0)
+    (property "Datasheet" "https://www.thegioiic.com/dien-tro-330-kohm-1-4w-5-4-vong-mau" (at 189.865 151.765 0)
       (effects (font (size 1.27 1.27)) hide)
     )
@@
     )
   )
+  (symbol (lib_id "power:GND1") (at 194.31 151.765 0) (unit 1)
+    (in_bom yes) (on_board yes) (dnp no)
+    (property "Reference" "#PWR046" (at 194.31 158.115 0)
+      (effects (font (size 1.27 1.27)) hide)
+    )
+    (property "Value" "GND1" (at 197.485 151.13 0)
+      (effects (font (size 1.27 1.27)))
+    )
+    (property "Footprint" "" (at 194.31 151.765 0)
+      (effects (font (size 1.27 1.27)) hide)
+    )
+    (property "Datasheet" "" (at 194.31 151.765 0)
+      (effects (font (size 1.27 1.27)) hide)
+    )
+    (pin "1")
+    (instances
+      (project "MACH_THUC"
+        (path "/fa9b692b-a58b-4246-a447-a74a2194b64e"
+          (reference "#PWR046") (unit 1)
+        )
+      )
+    )
+  )
   (symbol (lib_id "power:+5V") (at 107.95 154.94 90) (unit 1)
     (in_bom yes) (on_board yes) (dnp no) (fields_autoplaced)
@@
     )
   )
-  (symbol (lib_id "Device:R") (at 179.705 128.905 90) (unit 1)
+  (symbol (lib_id "Device:R") (at 178.435 128.905 90) (unit 1)
     (in_bom yes) (on_board yes) (dnp no) (fields_autoplaced)
-    (property "Reference" "R16" (at 179.705 122.555 90)
+    (property "Reference" "R16" (at 178.435 122.555 90)
       (effects (font (size 1.27 1.27)))
     )
-    (property "Value" "330" (at 179.705 125.095 90)
+    (property "Value" "330" (at 178.435 125.095 90)
       (effects (font (size 1.27 1.27)))
     )
-    (property "Footprint" "library_thuan_footprint:RES_DEFAULT" (at 179.705 130.683 90)
+    (property "Footprint" "library_thuan_footprint:RES_DEFAULT" (at 178.435 130.683 90)
       (effects (font (size 1.27 1.27)) hide)
     )
-    (property "Datasheet" "https://www.thegioiic.com/dien-tro-330-kohm-1-4w-5-4-vong-mau" (at 179.705 128.905 0)
+    (property "Datasheet" "https://www.thegioiic.com/dien-tro-330-kohm-1-4w-5-4-vong-mau" (at 178.435 128.905 0)
       (effects (font (size 1.27 1.27)) hide)
     )
@@
         )
       )
+    )
+  )
+  (symbol (lib_id "power:GND1") (at 182.88 128.905 0) (unit 1)
+    (in_bom yes) (on_board yes) (dnp no)
+    (property "Reference" "#PWR045" (at 182.88 135.255 0)
+      (effects (font (size 1.27 1.27)) hide)
+    )
+    (property "Value" "GND1" (at 186.055 128.27 0)
+      (effects (font (size 1.27 1.27)))
+    )
+    (property "Footprint" "" (at 182.88 128.905 0)
+      (effects (font (size 1.27 1.27)) hide)
+    )
+    (property "Datasheet" "" (at 182.88 128.905 0)
+      (effects (font (size 1.27 1.27)) hide)
+    )
+    (pin "1")
+    (instances
+      (project "MACH_THUC"
+        (path "/fa9b692b-a58b-4246-a447-a74a2194b64e"
+          (reference "#PWR045") (unit 1)
+        )
+      )

Commit message: update code'
Parts:
- U4: footprint library_thuan_footprint:PCF8574 -> library_thuan_footprint:SOIC127P1032X265-16N
Connections:
- net +5V: now also U3.15 (A/VEE)
- net rx: now also ESP_12E1.20 (D8); no longer ESP_12E1.18 (TX)
- net at R13.2, R14.1: now also ESP_12E1.21 (D7); no longer ESP_12E1.19 (RX)
- net at U4.7 (P3): no longer U3.15 (A/VEE)
- no-connect marks 2 -> 1
Other:
- moved on the sheet: R13, R14
Changed lines of the file:
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@@
   (junction (at 82.55 41.275) (diameter 0) (color 0 0 0 0)
   )
-  (junction (at 140.97 147.32) (diameter 0) (color 0 0 0 0)
-  )
   (junction (at 87.63 78.105) (diameter 0) (color 0 0 0 0)
   )
@@
   (junction (at 51.435 52.705) (diameter 0) (color 0 0 0 0)
   )
+  (junction (at 140.97 142.24) (diameter 0) (color 0 0 0 0)
+  )
   (junction (at 152.4 61.595) (diameter 0) (color 0 0 0 0)
   )
@@
   (junction (at 212.725 38.735) (diameter 0) (color 0 0 0 0)
   )
-  (no_connect (at 200.025 23.495))
   (no_connect (at 254.635 31.75))
   (wire (pts (xy 33.02 31.115) (xy 38.1 31.115))
@@
     (stroke (width 0) (type default))
   )
-  (wire (pts (xy 140.97 146.05) (xy 140.97 147.32))
+  (wire (pts (xy 140.97 141.605) (xy 140.97 142.24))
     (stroke (width 0) (type default))
   )
@@
     (stroke (width 0) (type default))
   )
+  (wire (pts (xy 140.97 142.24) (xy 140.97 144.145))
+    (stroke (width 0) (type default))
+  )
   (wire (pts (xy 49.53 131.445) (xy 49.53 138.43))
     (stroke (width 0) (type default))
@@
     (stroke (width 0) (type default))
   )
+  (wire (pts (xy 132.08 142.24) (xy 140.97 142.24))
+    (stroke (width 0) (type default))
+  )
   (wire (pts (xy 188.595 80.01) (xy 188.595 87.63))
     (stroke (width 0) (type default))
@@
     (stroke (width 0) (type default))
   )
+  (wire (pts (xy 133.985 144.78) (xy 132.08 144.78))
+    (stroke (width 0) (type default))
+  )
   (wire (pts (xy 243.205 109.855) (xy 243.205 121.285))
     (stroke (width 0) (type default))
@@
     (stroke (width 0) (type default))
   )
-  (wire (pts (xy 44.45 134.62) (xy 61.595 134.62))
-    (stroke (width 0) (type default))
-  )
   (wire (pts (xy 51.435 52.705) (xy 51.435 53.34))
     (stroke (width 0) (type default))
@@
     (stroke (width 0) (type default))
   )
-  (wire (pts (xy 133.35 149.86) (xy 132.08 149.86))
-    (stroke (width 0) (type default))
-  )
   (wire (pts (xy 236.855 21.59) (xy 236.855 26.035))
     (stroke (width 0) (type default))
@@
     (stroke (width 0) (type default))
   )
-  (wire (pts (xy 61.595 108.585) (xy 61.595 134.62))
-    (stroke (width 0) (type default))
-  )
   (wire (pts (xy 27.305 33.655) (xy 27.305 31.115))
     (stroke (width 0) (type default))
@@
     (stroke (width 0) (type default))
   )
-  (wire (pts (xy 140.97 147.32) (xy 140.97 148.59))
-    (stroke (width 0) (type default))
-  )
   (wire (pts (xy 29.21 138.43) (xy 29.21 131.445))
     (stroke (width 0) (type default))
@@
     (stroke (width 0) (type default))
   )
-  (wire (pts (xy 61.595 108.585) (xy 31.75 108.585))
-    (stroke (width 0) (type default))
-  )
   (wire (pts (xy 41.91 77.47) (xy 41.91 76.835))
     (stroke (width 0) (type default))
@@
     (stroke (width 0) (type default))
   )
-  (wire (pts (xy 44.45 138.43) (xy 44.45 134.62))
-    (stroke (width 0) (type default))
-  )
   (wire (pts (xy 34.29 111.125) (xy 36.195 111.125))
     (stroke (width 0) (type default))
@@
     (stroke (width 0) (type default))
   )
-  (wire (pts (xy 31.75 108.585) (xy 31.75 111.125))
-    (stroke (width 0) (type default))
-  )
   (wire (pts (xy 18.415 33.655) (xy 18.415 41.275))
     (stroke (width 0) (type default))
@@
   )
   (wire (pts (xy 104.14 38.735) (xy 104.14 41.275))
-    (stroke (width 0) (type default))
-  )
-  (wire (pts (xy 132.08 147.32) (xy 140.97 147.32))
     (stroke (width 0) (type default))
   )
@@
     )
   )
-  (global_label "tx" (shape input) (at 140.97 138.43 90) (fields_autoplaced)
+  (global_label "tx" (shape input) (at 140.97 133.985 90) (fields_autoplaced)
     (effects (font (size 1.27 1.27)) (justify left))
-    (property "Intersheetrefs" "${INTERSHEET_REFS}" (at 140.97 133.691 90)
+    (property "Intersheetrefs" "${INTERSHEET_REFS}" (at 140.97 129.246 90)
       (effects (font (size 1.27 1.27)) (justify left) hide)
     )
@@
     )
   )
-  (global_label "rx" (shape input) (at 133.35 149.86 0) (fields_autoplaced)
+  (global_label "rx" (shape input) (at 133.985 144.78 0) (fields_autoplaced)
     (effects (font (size 1.27 1.27)) (justify left))
-    (property "Intersheetrefs" "${INTERSHEET_REFS}" (at 138.1495 149.86 0)
+    (property "Intersheetrefs" "${INTERSHEET_REFS}" (at 138.7845 144.78 0)
       (effects (font (size 1.27 1.27)) (justify left) hide)
     )
@@
     )
   )
-  (symbol (lib_id "power:GND1") (at 140.97 156.21 0) (unit 1)
+  (symbol (lib_id "power:GND1") (at 140.97 151.765 0) (unit 1)
     (in_bom yes) (on_board yes) (dnp no)
-    (property "Reference" "#PWR034" (at 140.97 162.56 0)
-      (effects (font (size 1.27 1.27)) hide)
-    )
-    (property "Value" "GND1" (at 144.145 155.575 0)
-      (effects (font (size 1.27 1.27)))
-    )
-    (property "Footprint" "" (at 140.97 156.21 0)
-      (effects (font (size 1.27 1.27)) hide)
-    )
-    (property "Datasheet" "" (at 140.97 156.21 0)
+    (property "Reference" "#PWR034" (at 140.97 158.115 0)
+      (effects (font (size 1.27 1.27)) hide)
+    )
+    (property "Value" "GND1" (at 144.145 151.13 0)
+      (effects (font (size 1.27 1.27)))
+    )
+    (property "Footprint" "" (at 140.97 151.765 0)
+      (effects (font (size 1.27 1.27)) hide)
+    )
+    (property "Datasheet" "" (at 140.97 151.765 0)
       (effects (font (size 1.27 1.27)) hide)
     )
@@
       (effects (font (size 1.27 1.27)))
     )
-    (property "Footprint" "library_thuan_footprint:PCF8574" (at 46.99 151.13 0)
+    (property "Footprint" "library_thuan_footprint:SOIC127P1032X265-16N" (at 46.99 151.13 0)
       (effects (font (size 1.27 1.27)) hide)
     )
@@
     )
   )
-  (symbol (lib_id "Device:R") (at 140.97 142.24 0) (unit 1)
-    (in_bom yes) (on_board yes) (dnp no) (fields_autoplaced)
-    (property "Reference" "R13" (at 143.51 140.97 0)
-      (effects (font (size 1.27 1.27)) (justify left))
-    )
-    (property "Value" "1.2k" (at 143.51 143.51 0)
-      (effects (font (size 1.27 1.27)) (justify left))
-    )
-    (property "Footprint" "library_thuan_footprint:RES_DEFAULT" (at 139.192 142.24 90)
-      (effects (font (size 1.27 1.27)) hide)
-    )
-    (property "Datasheet" "https://www.thegioiic.com/dien-tro-1-2-kohm-1-4w-5-4-vong-mau" (at 140.97 142.24 0)
+  (symbol (lib_id "Device:R") (at 140.97 137.795 0) (unit 1)
+    (in_bom yes) (on_board yes) (dnp no) (fields_autoplaced)
+    (property "Reference" "R13" (at 143.51 136.525 0)
+      (effects (font (size 1.27 1.27)) (justify left))
+    )
+    (property "Value" "1.2k" (at 143.51 139.065 0)
+      (effects (font (size 1.27 1.27)) (justify left))
+    )
+    (property "Footprint" "library_thuan_footprint:RES_DEFAULT" (at 139.192 137.795 90)
+      (effects (font (size 1.27 1.27)) hide)
+    )
+    (property "Datasheet" "https://www.thegioiic.com/dien-tro-1-2-kohm-1-4w-5-4-vong-mau" (at 140.97 137.795 0)
       (effects (font (size 1.27 1.27)) hide)
     )
@@
         (path "/fa9b692b-a58b-4246-a447-a74a2194b64e"
           (reference "C2") (unit 1)
+        )
+      )
+    )
+  )
+  (symbol (lib_id "power:+5V") (at 31.75 111.125 90) (unit 1)
+    (in_bom yes) (on_board yes) (dnp no) (fields_autoplaced)
+    (property "Reference" "#PWR047" (at 35.56 111.125 0)
+      (effects (font (size 1.27 1.27)) hide)
+    )
+    (property "Value" "+5V" (at 28.575 111.125 90)
+      (effects (font (size 1.27 1.27)) (justify left))
+    )
+    (property "Footprint" "" (at 31.75 111.125 0)
+      (effects (font (size 1.27 1.27)) hide)
+    )
+    (property "Datasheet" "" (at 31.75 111.125 0)
+      (effects (font (size 1.27 1.27)) hide)
+    )
+    (pin "1")
+    (instances
+      (project "MACH_THUC"
+        (path "/fa9b692b-a58b-4246-a447-a74a2194b64e"
+          (reference "#PWR047") (unit 1)
         )
       )
@@
     )
   )
-  (symbol (lib_id "Device:R") (at 140.97 152.4 0) (unit 1)
-    (in_bom yes) (on_board yes) (dnp no) (fields_autoplaced)
-    (property "Reference" "R14" (at 143.51 151.13 0)
-      (effects (font (size 1.27 1.27)) (justify left))
-    )
-    (property "Value" "2.4k" (at 143.51 153.67 0)
-      (effects (font (size 1.27 1.27)) (justify left))
-    )
-    (property "Footprint" "library_thuan_footprint:RES_DEFAULT" (at 139.192 152.4 90)
-      (effects (font (size 1.27 1.27)) hide)
-    )
-    (property "Datasheet" "https://www.thegioiic.com/dien-tro-2-4-kohm-1-4w-1-5-vong-mau" (at 140.97 152.4 0)
-      (effects (font (size 1.27 1.27)) hide)
-    )
+  (symbol (lib_id "Device:R") (at 140.97 147.955 0) (unit 1)
+    (in_bom yes) (on_board yes) (dnp no) (fields_autoplaced)
+    (property "Reference" "R14" (at 143.51 146.685 0)
+      (effects (font (size 1.27 1.27)) (justify left))
+    )
+    (property "Value" "2.4k" (at 143.51 149.225 0)
+      (effects (font (size 1.27 1.27)) (justify left))
+    )
+    (property "Footprint" "library_thuan_footprint:RES_DEFAULT" (at 139.192 147.955 90)
+      (effects (font (size 1.27 1.27)) hide)
+    )
+    (property "Datasheet" "https://www.thegioiic.com/dien-tro-2-4-kohm-1-4w-1-5-vong-mau" (at 140.97 147.955 0)
+      (effects (font (size 1.27 1.27)) hide)
+    )

Commit message: update for finnal code
Parts:
- removed Q1: 2SB688, Package_TO_SOT_THT:TO-218-3_Vertical, symbol Transistor_BJT:2SB631
- removed R1, R2, R3: 100ohm, library_thuan_footprint:RES_1ohm_1w, symbol Device:R
Connections:
- net +5V: now also C3.1, C5.1, D1.2 (A), R4.1, U1.3 (VO); no longer D3.2 (A), R4.2
- net at B1.2 (VIN), C6.1, SS1.2 (S3): now also C2.1, C4.1, D1.1 (K), U1.1 (VI)
- new net: D3.2 (A), R4.2
Other:
- moved on the sheet: B1, C10, C2, C3, C4, C5, C6, C7, D1, D3, PB1, PB2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
