File: PROJECT/MACH/MACH_THUC/MACH_THUC/MACH_THUC_V2/MACH_THUC_V2/MACH_THUC_V2.kicad_pcb (KiCad board)
At the start: 2 copper layers, 104.1 x 73.7 mm, 22 parts, among them J1 1935161, U1 L7805, Y1 Crystal 20M

Commit message: update code
Connections:
- S1 pad S1: unconnected-(S1-SHIELD-PadS1) -> unconnected-(S1-SHIELD-PadS1)_0
