File: PROJECT/MACH/MACH_THUC/MACH_THUC/MACH_THUC_V2/MACH_THUC_V2/MACH_THUC_V2.kicad_sch (KiCad schematic)
At the start: 22 parts, among them J1 1935161, U1 L7805, Y1 Crystal 20M

Commit message: update code final
Parts:
- added DS1: WC1602A, Display:WC1602A, symbol Display_Character:WC1602A
Changed lines of the file:
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@@
+	)
+	(symbol
+		(lib_id "Display_Character:WC1602A")
+		(at 49.53 114.3 0)
+		(unit 1)
+		(exclude_from_sim no)
+		(in_bom yes)
+		(on_board yes)
+		(dnp no)
+		(fields_autoplaced yes)
+		(property "Reference" "DS1"
+			(at 51.7241 91.44 0)
+			(effects
+				(font
+					(size 1.27 1.27)
+				)
+				(justify left)
+			)
+		)
+		(property "Value" "WC1602A"
+			(at 51.7241 93.98 0)
+			(effects
+				(font
+					(size 1.27 1.27)
+				)
+				(justify left)
+			)
+		)
+		(property "Footprint" "Display:WC1602A"
+			(at 49.53 137.16 0)
+			(effects
+				(font
+					(size 1.27 1.27)
+					(italic yes)
+				)
+				(hide yes)
+			)
+		)
+		(property "Datasheet" "http://www.wincomlcd.com/pdf/WC1602A-SFYLYHTC06.pdf"
+			(at 67.31 114.3 0)
+			(effects
+				(font
+					(size 1.27 1.27)
+				)
+				(hide yes)
+			)
+		)
+		(property "Description" "LCD 16x2 Alphanumeric , 8 bit parallel bus, 5V VDD"
+			(at 49.53 114.3 0)
+			(effects
+				(font
+					(size 1.27 1.27)
+				)
+				(hide yes)
+			)
+		)
+		(pin "15"
+		)
+		(pin "12"
+		)
+		(pin "1"
+		)
+		(pin "7"
+		)
+		(pin "10"
+		)
+		(pin "16"
+		)
+		(pin "8"
+		)
+		(pin "9"
+		)
+		(pin "13"
+		)
+		(pin "5"
+		)
+		(pin "2"
+		)
+		(pin "14"
+		)
+		(pin "3"
+		)
+		(pin "4"
+		)
+		(pin "6"
+		)
+		(pin "11"
+		)
+		(instances
+			(project "MACH_THUC_V2"
+				(path "/5e179f03-c6e4-4dcc-af17-ffe7add0ada4"
+					(reference "DS1")
+					(unit 1)
+				)
+			)
+		)
 	)
 	(symbol
